Commit message: Update

File: tf_urdf2/urdf/tf_urdf2.urdf (robot description, URDF)
Before this commit: robot tf_urdf2, 13 links, 12 joints
Links:
- added link base_footprint
Joints:
- added joint base_joint: type fixed, parent base_footprint, child base_link, origin xyz=-1.23025786656509E-12 5.18846734977975E-12 7.17791849942659E-12 rpy=0 0 0
