Commit message: Config package to launch fullsystem

File: tf_urdf3/urdf/tf_urdf3.urdf (robot description, URDF)
Before this commit: robot tf_urdf3, 12 links, 11 joints
Links:
- added link base_footprint
Joints:
- added joint base_joint: type fixed, parent base_footprint, child base_link, origin xyz=-1.05559497177638E-12 6.31894336221611E-12 -5.17741961678007E-12 rpy=0 0 0
