Commit message: Add base_footprint

File: tf_urdf4/urdf/tf_urdf4.urdf (robot description, URDF)
Before this commit: robot tf_urdf4, 12 links, 11 joints
Links:
- added link base_footprint
Joints:
- added joint base_joint: type fixed, parent base_footprint, child base_link, origin xyz=-1.05560534986818E-12 5.17741757590009E-12 6.3189360698697E-12 rpy=0 0 0

Commit message: Config URDF coordinate

File: tf_urdf4/urdf/tf_urdf4.urdf (robot description, URDF)
Before this commit: robot tf_urdf4, 13 links, 12 joints
Joints:
- joint scan_joint: origin xyz=-0.000111983196857368 0.0672432860074702 0.0279411844683552 rpy=0 0 1.5707963267949 -> xyz=-0.000111983196857368 0.0672432860074702 0.0279411844683552 rpy=0 0 -1.507

Commit message: Config lidar angle, apply laser_scan to full_launch.launch and config URDF base_scan frame to same with real world angle

File: tf_urdf4/urdf/tf_urdf4.urdf (robot description, URDF)
Before this commit: robot tf_urdf4, 13 links, 12 joints
Joints:
- joint scan_joint: origin xyz=-0.000111983196857368 0.0672432860074702 0.0279411844683552 rpy=0 0 -1.507 -> xyz=-0.000111983196857368 0.0672432860074702 0.0279411844683552 rpy=0 0 -1.66
