Commit message: Update launch file tf_urdf

File: nav_tf_urdf/urdf/nav_tf_urdf.urdf (robot description, URDF)
Before this commit: robot nav_tf_urdf, 6 links, 5 joints
Joints:
- joint scan_joint: origin xyz=0 0.0120740335852946 0.0743670768316607 rpy=-1.5707963267949 0 -1.5707963267949 -> xyz=0 0.0120740335852946 0.0743670768316607 rpy=0 0 -1.5707963267949

Commit message: Update nav_tf_urdf.urdf

File: nav_tf_urdf/urdf/nav_tf_urdf.urdf (robot description, URDF)
Before this commit: robot nav_tf_urdf, 6 links, 5 joints
Joints:
- joint scan_joint: axis 0 1 0 -> 0 0 1

Commit message: Update nav_tf_urdf.urdf

File: nav_tf_urdf/urdf/nav_tf_urdf.urdf (robot description, URDF)
Before this commit: robot nav_tf_urdf, 6 links, 5 joints
Joints:
- joint scan_joint: axis 0 0 1 -> 0 1 0
